File: schematic.sch (EAGLE design)
At the start: 7 parts

Commit message: Improved schematic file
Parts:
- removed PWR: (no value), con-wago-500:W237-102
- added J1: POWER_JACK, SparkFun-Connectors:POWER_JACK
Connections:
- net LPWM renamed M1_LEFT_PWM
- net N$7 renamed BT_TX
- net N$8 renamed BT_RX
- net RPWM renamed M1_RIGHT_PWM
- removed net N$1: U$1.D2, U$3.D3
- removed net N$2: U$1.D3, U$3.D2
- removed net N$3: U$1.D4, U$2.D3
- removed net N$4: U$1.D5, U$2.D2
- removed net N$5: MOTOR2.1, U$3.D9
- removed net N$6: MOTOR2.2, U$3.D10
- new net M2_LEFT_PWM: MOTOR2.2, U$3.D9
- new net M2_RIGHT_PWM: MOTOR2.1, U$3.D10
- new net SLAVE1_RX: U$1.D3, U$2.D2
- new net SLAVE1_TX: U$1.D2, U$2.D3
- new net SLAVE2_RX: U$1.D5, U$3.D2
- new net SLAVE2_TX: U$1.D4, U$3.D3
- net GND: now also J1.GND, J1.GNDBREAK; no longer PWR-1.KL
- net VCC: now also J1.PWR; no longer PWR-2.KL
Other:
- note added: "BLUETOOTH"
- note added: "MASTER ARDUINO"
- note added: "MOTOR CONNECTIONS"
- note added: "POWER"
- note added: "SLAVE ARDUINOS"
- moved on the sheet: HC06, MOTOR1, MOTOR2

Commit message: edit
Parts:
- removed HC06: (no value), pinhead:PINHD-1X4
- removed J1: POWER_JACK, SparkFun-Connectors:POWER_JACK
- added BT: HC06_BLUETOOTH, OnurLibrary:HC06_BLUETOOTH
- added X1: (no value), con-wago-500:W237-102
Connections:
- new net 5V: BT.VCC, MOTOR1.3, MOTOR1.4, MOTOR1.7, MOTOR2.3, MOTOR2.4, MOTOR2.7, U$2.5.5V
- net BT_RX: now also BT.RX; no longer HC06.1
- net BT_TX: now also BT.TX; no longer HC06.2
- net GND: now also BT.GND, U$1.GND2, U$2.GND2, U$3.GND2, X1-2.KL; no longer HC06.3, J1.GND, J1.GNDBREAK, U$1.GND
- net M1_LEFT_PWM: now also U$2.D10; no longer U$2.D9
- net M1_RIGHT_PWM: now also U$2.D9; no longer U$2.D10
- net M2_LEFT_PWM: now also U$3.D10; no longer U$3.D9
- net M2_RIGHT_PWM: now also U$3.D9; no longer U$3.D10
- net VCC: now also X1-1.KL; no longer HC06.4, J1.PWR, MOTOR1.3, MOTOR1.4, MOTOR1.7, MOTOR2.3, MOTOR2.4, MOTOR2.7
