File: schematic.brd (EAGLE design)
At the start: 92.7 x 74.6 mm, 7 parts

Commit message: edit
Connections:
- net 5V: no longer U$3.5V
Changed lines of the file:
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@@
 <contactref element="BT" pad="VCC"/>
 <contactref element="U$2" pad="5V"/>
-<contactref element="U$3" pad="5V"/>
 <wire x1="11.43" y1="38.1" x2="11.43" y2="40.64" width="0.1524" layer="16"/>
 <wire x1="11.43" y1="40.64" x2="8.89" y2="43.18" width="0.1524" layer="16"/>
@@
 <wire x1="38.1" y1="59.69" x2="45.72" y2="59.69" width="0.1524" layer="16"/>
 <wire x1="45.72" y1="59.69" x2="49.53" y2="63.5" width="0.1524" layer="16"/>
-<wire x1="11.43" y1="38.1" x2="33.02" y2="15.24" width="0" layer="19" extent="1-1"/>
 </signal>
 <signal name="N$2">

Commit message: Board updated
Other:
- board size 92.7 x 74.6 mm -> 95.2 x 68.2 mm

Commit message: Board updated
Routing:
- net VCC: track 187.4 -> 119.6 mm
- net GND: track 199.1 -> 210.0 mm
- net BT_TX: track 51.3 -> 54.3 mm
- net SLAVE1_RX: track 36.5 -> 38.7 mm
- net M1_RIGHT_PWM: track 8.98 -> 11.2 mm
- net SLAVE2_TX: track 25.5 -> 27.7 mm
- net 5V: track 104.3 -> 106.0 mm
- net SLAVE2_RX: track 21.9 -> 23.4 mm
- net M1_LEFT_PWM: track 14.1 -> 15.5 mm
- net M2_RIGHT_PWM: track 12.8 -> 14.3 mm
- net SLAVE1_TX: track 32.8 -> 34.3 mm
- net M2_LEFT_PWM: track 9.20 -> 9.94 mm
Other:
- board size 95.2 x 68.2 mm -> 72.4 x 68.2 mm

Commit message: Trace updated
Routing:
- net SLAVE1_TX: track 34.3 -> 35.7 mm
Changed lines of the file:
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@@
 <wire x1="34.29" y1="53.34" x2="38.1" y2="49.53" width="0.381" layer="16"/>
 <wire x1="38.1" y1="49.53" x2="43.18" y2="49.53" width="0.381" layer="16"/>
-<wire x1="43.18" y1="49.53" x2="50.8" y2="41.91" width="0.381" layer="16"/>
 <wire x1="34.29" y1="55.88" x2="31.75" y2="58.42" width="0.381" layer="16"/>
 <wire x1="31.75" y1="58.42" x2="29.21" y2="58.42" width="0.381" layer="16"/>
 <wire x1="29.21" y1="58.42" x2="27.94" y2="59.69" width="0.381" layer="16"/>
 <wire x1="27.94" y1="59.69" x2="27.94" y2="62.23" width="0.381" layer="16"/>
+<wire x1="43.18" y1="49.53" x2="45.72" y2="46.99" width="0.381" layer="16"/>
+<wire x1="45.72" y1="46.99" x2="45.72" y2="44.45" width="0.381" layer="16"/>
+<wire x1="45.72" y1="44.45" x2="48.26" y2="41.91" width="0.381" layer="16"/>
+<wire x1="48.26" y1="41.91" x2="50.8" y2="41.91" width="0.381" layer="16"/>
 </signal>
 <signal name="SLAVE2_RX">

Commit message: Board updated
Routing:
- net SLAVE1_TX: track 35.7 -> 34.3 mm
- net GND: track 210.0 -> 208.9 mm
Other:
- board text added: "PWM Control Circuit"

Commit message: Changes for production
Other:
- board size 72.4 x 68.2 mm -> 73.7 x 68.6 mm
- board text added: "O.S."
Changed lines of the file:
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@@
 <setting verticaltext="up"/>
 </settings>
-<grid distance="1" unitdist="mil" unit="mil" style="lines" multiple="1" display="yes" altdistance="5" altunitdist="mil" altunit="mil"/>
+<grid distance="1" unitdist="mm" unit="mm" style="lines" multiple="1" display="yes" altdistance="0.05" altunitdist="inch" altunit="inch"/>
 <layers>
 <layer number="1" name="Top" color="4" fill="1" visible="yes" active="yes"/>
@@
 <layer number="43" name="vRestrict" color="2" fill="10" visible="yes" active="yes"/>
 <layer number="44" name="Drills" color="7" fill="1" visible="no" active="yes"/>
-<layer number="45" name="Holes" color="7" fill="1" visible="no" active="yes"/>
+<layer number="45" name="Holes" color="7" fill="1" visible="yes" active="yes"/>
 <layer number="46" name="Milling" color="3" fill="1" visible="no" active="yes"/>
 <layer number="47" name="Measures" color="7" fill="1" visible="no" active="yes"/>
@@
 <board>
 <plain>
-<wire x1="-2.54" y1="8.89" x2="69.83" y2="8.89" width="0" layer="20"/>
-<wire x1="69.83" y1="8.89" x2="69.83" y2="77.14" width="0" layer="20"/>
-<wire x1="69.83" y1="77.14" x2="-2.54" y2="77.14" width="0" layer="20"/>
-<wire x1="-2.54" y1="77.14" x2="-2.54" y2="8.89" width="0" layer="20"/>
+<wire x1="-2.54" y1="7.62" x2="71.12" y2="7.62" width="0" layer="20"/>
+<wire x1="71.12" y1="7.62" x2="71.12" y2="76.2" width="0" layer="20"/>
+<wire x1="71.12" y1="76.2" x2="-2.54" y2="76.2" width="0" layer="20"/>
+<wire x1="-2.54" y1="76.2" x2="-2.54" y2="7.62" width="0" layer="20"/>
 <rectangle x1="25.0571" y1="35.0647" x2="25.0825" y2="35.0901" layer="21"/>
 <rectangle x1="25.0317" y1="35.1155" x2="25.1079" y2="35.1409" layer="21"/>
@@
 <rectangle x1="25.0063" y1="41.8465" x2="25.1333" y2="41.8719" layer="21"/>
 <rectangle x1="25.0571" y1="41.8719" x2="25.0825" y2="41.8973" layer="21"/>
-<text x="52.6796" y="9.9314" size="1.27" layer="21" font="vector">PWM Control Circuit</text>
+<text x="48.8696" y="8.6614" size="1.27" layer="21" font="vector">PWM Control Circuit</text>
+<hole x="0" y="73.66" drill="3.5"/>
+<hole x="68.58" y="73.66" drill="3.5"/>
+<hole x="68.58" y="10.16" drill="3.5"/>
+<hole x="0" y="10.16" drill="3.5"/>
+<text x="8" y="9" size="1.778" layer="22" rot="MR0">O.S.</text>
 </plain>
 <attributes>
